File: simulations/parallel_discharge/parallel_discharge.kicad_sch (KiCad schematic)
At the start: 9 parts

Commit message: More simulations :)
Parts:
- R1, R2, R3, R4, R7: value 470 -> 1k
Changed lines of the file:
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@@
 			)
 		)
-		(property "Value" "470"
+		(property "Value" "1k"
 			(at 104.14 80.0099 0)
 			(show_name no)
@@
 			)
 		)
-		(property "Value" "470"
+		(property "Value" "1k"
 			(at 90.17 80.0099 0)
 			(show_name no)
@@
 			)
 		)
-		(property "Value" "470"
+		(property "Value" "1k"
 			(at 118.11 80.0099 0)
 			(show_name no)
@@
 			)
 		)
-		(property "Value" "470"
+		(property "Value" "1k"
 			(at 76.2 80.0099 0)
 			(show_name no)
@@
 			)
 		)
-		(property "Value" "470"
+		(property "Value" "1k"
 			(at 132.08 88.8999 0)
 			(show_name no)
